File: BLE_sensors_pcb/design_files/Accelerometer-Magnetometer.kicad_sch (KiCad schematic)
At the start: 5 parts, among them U2 LSM303AHTR

Commit message: Added pdf
Changed lines of the file:
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@@
 	(text "Accelerometer Magnetometer\n"
 		(exclude_from_sim no)
-		(at 145.034 42.926 0)
+		(at 145.542 78.232 0)
 		(effects
 			(font
