File: BLE_sensors_pcb/design_files/Temp_Sensor.kicad_sch (KiCad schematic)
At the start: 5 parts, among them U1 BME280

Commit message: Added pdf
Changed lines of the file:
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@@
 	(text "Temp Sensor\n"
 		(exclude_from_sim no)
-		(at 140.97 37.338 0)
+		(at 138.43 66.802 0)
 		(effects
 			(font
