File: BLE_sensors_pcb/design_files/USB_to_Serial.kicad_sch (KiCad schematic)
At the start: 5 parts, among them U7 MCP2221AxST

Commit message: Added pdf
Changed lines of the file:
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@@
 	(text "USB to Serial\n"
 		(exclude_from_sim no)
-		(at 145.288 35.306 0)
+		(at 146.558 71.374 0)
 		(effects
 			(font
